Commit message: added all gazebo plugins and initialized navigation pacakage

File: src/stembotx2_description/urdf/stembotx2.xacro.urdf (robot description, URDF)
Before this commit: robot stembotx2, 12 links, 11 joints
Links:
- added link base_footprint
- link Agv_back_castor_wheel_link_1: mass 0.02104448198884657 -> 0.3
- link Agv_front_castor_wheel_link_1: mass 0.02104448198884657 -> 0.3
- link Agv_left_wheel_link_1: mass 0.6042068071016569 -> 1
- link Agv_right_wheel_link_1: mass 0.6042068071016568 -> 1
- link base_link: mass 113.06787878589044 -> 10
Joints:
- removed joint Revolute 6
- removed joint Revolute 7
- added joint base_footprint_joint: type fixed, parent base_footprint, child base_link, origin xyz=0 0 0.0175 rpy=0 0 0
- added joint left_wheel_joint: type continuous, parent base_link, child Agv_left_wheel_link_1, origin xyz=0.081 0.0 0.035 rpy=0 0 0, axis 0.0 1.0 0.0
- added joint right_wheel_joint: type continuous, parent base_link, child Agv_right_wheel_link_1, origin xyz=-0.082 0.0 0.035 rpy=0 0 0, axis 0.0 1.0 0.0

Commit message: changed base footprint

File: src/stembotx2_description/urdf/stembotx2.xacro.urdf (robot description, URDF)
Before this commit: robot stembotx2, 13 links, 12 joints
Joints:
- joint base_footprint_joint: origin xyz=0 0 0.0175 rpy=0 0 0 -> xyz=0 0 0 rpy=0 0 0

Commit message: changed mass values

File: src/stembotx2_description/urdf/stembotx2.xacro.urdf (robot description, URDF)
Before this commit: robot stembotx2, 13 links, 12 joints
Links:
- link Agv_back_castor_wheel_link_1: mass 0.3 -> 0.5
- link Agv_front_castor_wheel_link_1: mass 0.3 -> 0.5
- link Agv_left_wheel_link_1: mass 1 -> 1.5
- link Agv_right_wheel_link_1: mass 1 -> 1.5
- link base_link: mass 10 -> 30
Joints:
- removed joint Rigid 8
- removed joint Rigid 9
- added joint back_castor_joint: type fixed, parent base_link, child Agv_back_castor_wheel_link_1, origin xyz=0.0 0.135 0.031 rpy=0 0 0
- added joint front_castor_joint: type fixed, parent base_link, child Agv_front_castor_wheel_link_1, origin xyz=0.0 -0.135 0.031 rpy=0 0 0
- joint base_footprint_joint: origin xyz=0 0 0 rpy=0 0 0 -> xyz=0 0 0.035 rpy=0 0 0
